File: kicad/distrib/distrib.sch (KiCad schematic (older format))
At the start: 35 parts, among them J1 Conn_01x03_Male, J10 Conn_01x03_Male, J11 Conn_01x03_Male, J12 Conn_01x03_Male, J13 Conn_01x03_Male, J14 Conn_01x03_Male, J15 Conn_01x03_Male, J16 Conn_01x03_Male, J17 Conn_01x03_Male, J18 Conn_01x03_Male, J19 Conn_01x03_Male, J2 Conn_01x03_Male, J20 Conn_01x03_Male, J21 Conn_01x03_Male, J22 Conn_01x03_Male, J23 Conn_01x03_Male, J24 Conn_01x03_Male, J25 Conn_01x03_Male, J26 Conn_01x03_Male, J27 Conn_01x03_Male, J28 Conn_01x03_Male, J29 Conn_01x03_Male, J3 Conn_01x03_Male, J30 Conn_01x03_Male, J31 Screw_Terminal_01x02, J4 Conn_01x03_Male, J5 Conn_01x03_Male, J6 Conn_01x03_Male, J7 Conn_01x03_Male, J8 Conn_01x03_Male, J9 Conn_01x03_Male

Commit message: autosave
Other:
- moved on the sheet: J31
Changed lines of the file:
@@
 L Connector:Screw_Terminal_01x02 J31
 U 1 1 5F74C7DE
-P 1500 3550
-F 0 "J31" H 1580 3542 50  0000 L CNN
-F 1 "Screw_Terminal_01x02" H 1580 3451 50  0000 L CNN
-F 2 "Connectors_Molex:Molex_KK-6410-02_02x2.54mm_Straight" H 1500 3550 50  0001 C CNN
-F 3 "~" H 1500 3550 50  0001 C CNN
-	1    1500 3550
+P 1150 3000
+F 0 "J31" H 1230 2992 50  0000 L CNN
+F 1 "Screw_Terminal_01x02" H 1230 2901 50  0000 L CNN
+F 2 "Connectors_Molex:Molex_KK-6410-02_02x2.54mm_Straight" H 1150 3000 50  0001 C CNN
+F 3 "~" H 1150 3000 50  0001 C CNN
+	1    1150 3000
 	1    0    0    -1
 $EndComp
@@
 L power:GND #PWR0103
 U 1 1 5F7AF352
-P 900 1050
-F 0 "#PWR0103" H 900 800 50  0001 C CNN
-F 1 "GND" H 905 877 50  0000 C CNN
-F 2 "" H 900 1050 50  0001 C CNN
-F 3 "" H 900 1050 50  0001 C CNN
-	1    900  1050
+P 650 650
+F 0 "#PWR0103" H 650 400 50  0001 C CNN
+F 1 "GND" H 655 477 50  0000 C CNN
+F 2 "" H 650 650 50  0001 C CNN
+F 3 "" H 650 650 50  0001 C CNN
+	1    650  650
 	1    0    0    -1
 $EndComp
@@
 L power:+12V #PWR0165
 U 1 1 5F7F2BAD
-P 1300 3550
-F 0 "#PWR0165" H 1300 3400 50  0001 C CNN
-F 1 "+12V" V 1315 3678 50  0000 L CNN
-F 2 "" H 1300 3550 50  0001 C CNN
-F 3 "" H 1300 3550 50  0001 C CNN
-	1    1300 3550
+P 950 3000
+F 0 "#PWR0165" H 950 2850 50  0001 C CNN
+F 1 "+12V" V 965 3128 50  0000 L CNN
+F 2 "" H 950 3000 50  0001 C CNN
+F 3 "" H 950 3000 50  0001 C CNN
+	1    950  3000
 	0    -1   -1   0
 $EndComp
@@
 L power:GND #PWR0166
 U 1 1 5F7F3A5F
-P 1300 3650
-F 0 "#PWR0166" H 1300 3400 50  0001 C CNN
-F 1 "GND" V 1305 3522 50  0000 R CNN
-F 2 "" H 1300 3650 50  0001 C CNN
-F 3 "" H 1300 3650 50  0001 C CNN
-	1    1300 3650
-	0    1    1    0
-$EndComp
+P 950 3100
+F 0 "#PWR0166" H 950 2850 50  0001 C CNN
+F 1 "GND" V 955 2972 50  0000 R CNN
+F 2 "" H 950 3100 50  0001 C CNN
+F 3 "" H 950 3100 50  0001 C CNN
+	1    950  3100
+	0    1    1    0
+$EndComp

Commit message: breakout
Parts:
- added J31, J32, J33: Conn_01x03_Male, Connectors_Phoenix:PhoenixContact_MCV-G_03x3.81mm_Vertical, symbol Connector:Conn_01x03_Male
- J1, J10, J11, J12, J13, J14, J15, J16, J17, J18, J19, J2, J20, J21, J22, J23, J24, J25, J26, J27, J28, J29, J3, J30, J4, J5, J6, J7, J8, J9: footprint Connectors_Molex:Molex_KK-6410-03_03x2.54mm_Straight -> Connectors_Phoenix:PhoenixContact_MCV-G_03x3.81mm_Vertical
- POWER1: renamed from J31; footprint Connectors_Molex:Molex_KK-6410-02_02x2.54mm_Straight -> Connector_AMASS:AMASS_XT60-F_1x02_P7.20mm_Vertical
Connections:
- net +12V: now also J31.1 (Pin_1), J32.1 (Pin_1), J33.1 (Pin_1)
- net GND: now also J31.3 (Pin_3), J32.3 (Pin_3), J33.3 (Pin_3)
- net at J30.2 (Pin_2): now also J31.2 (Pin_2)
- new net: J32.2 (Pin_2), J33.2 (Pin_2)
Other:
- moved on the sheet: H1, H2, H3, H4, POWER1

Commit message: distrib: ajout connecteur leds
Parts:
- added J34: LEDS, Pin_Headers:Pin_Header_Straight_1x03_Pitch2.54mm, symbol Connector_Generic:Conn_01x03
- added R1: 470, Resistors_SMD:R_0805_HandSoldering, symbol Device:R
- POWER1: value Screw_Terminal_01x02 -> XT60
Connections:
- net +12V: now also POWER1.2 (Pin_2); no longer POWER1.1 (Pin_1)
- net DATA_IN: now also R1.2
- net GND: now also POWER1.1 (Pin_1), J34.3 (Pin_3); no longer POWER1.2 (Pin_2)
- new net: J34.2 (Pin_2), R1.1
- no-connect marks 0 -> 1
Changed lines of the file:
@@
 P 1850 3950
 F 0 "POWER1" H 1930 3942 50  0000 L CNN
-F 1 "Screw_Terminal_01x02" H 1930 3851 50  0000 L CNN
+F 1 "XT60" H 1930 3851 50  0000 L CNN
 F 2 "Connector_AMASS:AMASS_XT60-F_1x02_P7.20mm_Vertical" H 1850 3950 50  0001 C CNN
 F 3 "~" H 1850 3950 50  0001 C CNN
@@
 L power:+12V #PWR071
 U 1 1 5F7F2BAD
+P 1650 4050
+F 0 "#PWR071" H 1650 3900 50  0001 C CNN
+F 1 "+12V" V 1665 4178 50  0000 L CNN
+F 2 "" H 1650 4050 50  0001 C CNN
+F 3 "" H 1650 4050 50  0001 C CNN
+	1    1650 4050
+	0    -1   -1   0
+$EndComp
+$Comp
+L power:GND #PWR072
+U 1 1 5F7F3A5F
 P 1650 3950
-F 0 "#PWR071" H 1650 3800 50  0001 C CNN
-F 1 "+12V" V 1665 4078 50  0000 L CNN
+F 0 "#PWR072" H 1650 3700 50  0001 C CNN
+F 1 "GND" V 1655 3822 50  0000 R CNN
 F 2 "" H 1650 3950 50  0001 C CNN
 F 3 "" H 1650 3950 50  0001 C CNN
 	1    1650 3950
-	0    -1   -1   0
-$EndComp
-$Comp
-L power:GND #PWR072
-U 1 1 5F7F3A5F
-P 1650 4050
-F 0 "#PWR072" H 1650 3800 50  0001 C CNN
-F 1 "GND" V 1655 3922 50  0000 R CNN
-F 2 "" H 1650 4050 50  0001 C CNN
-F 3 "" H 1650 4050 50  0001 C CNN
-	1    1650 4050
 	0    1    1    0
 $EndComp
@@
 Wire Wire Line
 	1700 1550 1350 1550
+$Comp
+L Connector_Generic:Conn_01x03 J34
+U 1 1 5F7990C4
+P 3650 4000
+F 0 "J34" H 3730 4042 50  0000 L CNN
+F 1 "LEDS" H 3730 3951 50  0000 L CNN
+F 2 "Pin_Headers:Pin_Header_Straight_1x03_Pitch2.54mm" H 3650 4000 50  0001 C CNN
+F 3 "~" H 3650 4000 50  0001 C CNN
+	1    3650 4000
+	1    0    0    -1
+$EndComp
+$Comp
+L power:GND #PWR0101
+U 1 1 5F79A69B
+P 3450 4100
+F 0 "#PWR0101" H 3450 3850 50  0001 C CNN
+F 1 "GND" V 3455 3972 50  0000 R CNN
+F 2 "" H 3450 4100 50  0001 C CNN
+F 3 "" H 3450 4100 50  0001 C CNN
+	1    3450 4100
+	0    1    1    0
+$EndComp
+Text GLabel 3050 4000 0    50   Input ~ 0
+DATA_IN
+NoConn ~ 3450 3900
+$Comp
+L Device:R R1
+U 1 1 5F7D0FC2
+P 3250 4000
+F 0 "R1" V 3043 4000 50  0000 C CNN
+F 1 "470" V 3134 4000 50  0000 C CNN
+F 2 "Resistors_SMD:R_0805_HandSoldering" V 3180 4000 50  0001 C CNN
+F 3 "~" H 3250 4000 50  0001 C CNN
+	1    3250 4000
+	0    1    1    0
+$EndComp
+Wire Wire Line
+	3100 4000 3050 4000
+Wire Wire Line
+	3400 4000 3450 4000
 $EndSCHEMATC
