File: kicad/distrilite/distrilite.sch (KiCad schematic (older format))
At the start: 25 parts, among them J1 Conn_01x03_Male, J10 Conn_01x03_Male, J11 Conn_01x03_Male, J12 Conn_01x03_Male, J13 LED_DOUT, J2 Conn_01x03_Male, J3 Conn_01x03_Male, J34 LED_DIN, J4 Conn_01x03_Male, J5 Conn_01x03_Male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

Commit message: ajout condo et validation ?
Parts:
- added C1, C2: CP, Capacitors_ThroughHole:CP_Radial_D10.0mm_P3.80mm, symbol Device:CP
- H1, H2, H3, H4: footprint Mounting_Holes:MountingHole_3.2mm_M3 -> Mounting_Holes:MountingHole_3.2mm_M3_Pad
Connections:
- net +12V: now also C1.1, C2.1
- net GND: now also C1.2, C2.2
Other:
- moved on the sheet: H1, H2, H3, H4, J1, J10, J11, J12, J13, J2, J3, J34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
