File: kicad/espbreakout/espbreakout.sch (KiCad schematic (older format))
At the start: 18 parts, among them J1 TEMPERATURE, J2 POWER, J3 CURRENT, J4 LED DATA, J5 RELAY, J6 Conn_01x19, J7 Conn_01x19, J8 I2C, J9 SERIAL

Commit message: esp breakout board (wip)
Parts:
- added D?: RELAY, LED_SMD:LED_1206_3216Metric_Pad1.42x1.75mm_HandSolder, symbol Device:LED
- added JP?: PLJP, Jumper:SolderJumper-2_P1.3mm_Open_RoundedPad1.0x1.5mm, symbol Jumper:SolderJumper_2_Open
- added R?: 51, Resistors_SMD:R_0805_HandSoldering, symbol Device:R
- R3: value 330 -> 150
Connections:
- net GND: now also D?.1 (K)
- net RELAI_TRIGGER renamed RELAY_TRIGGER
- net RELAY_TRIGGER: now also JP?.2 (B)
- new net: D?.2 (A), R?.2
- new net: JP?.1 (A), R?.1
Other:
- moved on the sheet: D1, JP1, R3
Changed lines of the file:
@@
 EESchema Schematic File Version 4
+LIBS:espbreakout-cache
 EELAYER 30 0
 EELAYER END
@@
 CURRENT_SENSOR
 Text GLabel 5900 3550 0    50   Output ~ 0
-RELAI_TRIGGER
+RELAY_TRIGGER
 Text GLabel 1250 3100 2    50   Output ~ 0
 LED_DATA
@@
 L Device:LED D1
 U 1 1 5FB11385
-P 4050 1250
-F 0 "D1" H 4043 1466 50  0000 C CNN
-F 1 "POWER" H 4043 1375 50  0000 C CNN
-F 2 "LED_SMD:LED_1206_3216Metric_Pad1.42x1.75mm_HandSolder" H 4050 1250 50  0001 C CNN
-F 3 "~" H 4050 1250 50  0001 C CNN
-	1    4050 1250
+P 4000 1100
+F 0 "D1" H 3993 1316 50  0000 C CNN
+F 1 "POWER" H 3993 1225 50  0000 C CNN
+F 2 "LED_SMD:LED_1206_3216Metric_Pad1.42x1.75mm_HandSolder" H 4000 1100 50  0001 C CNN
+F 3 "~" H 4000 1100 50  0001 C CNN
+	1    4000 1100
 	1    0    0    -1
 $EndComp
@@
 L Jumper:SolderJumper_2_Open JP1
 U 1 1 5FB12326
-P 4650 1250
-F 0 "JP1" H 4650 1363 50  0000 C CNN
-F 1 "PLJP" H 4650 1364 50  0001 C CNN
-F 2 "Jumper:SolderJumper-2_P1.3mm_Open_RoundedPad1.0x1.5mm" H 4650 1250 50  0001 C CNN
-F 3 "~" H 4650 1250 50  0001 C CNN
-	1    4650 1250
+P 4600 1100
+F 0 "JP1" H 4600 1213 50  0000 C CNN
+F 1 "PLJP" H 4600 1214 50  0001 C CNN
+F 2 "Jumper:SolderJumper-2_P1.3mm_Open_RoundedPad1.0x1.5mm" H 4600 1100 50  0001 C CNN
+F 3 "~" H 4600 1100 50  0001 C CNN
+	1    4600 1100
 	1    0    0    -1
 $EndComp
@@
 L power:+5V #PWR0123
 U 1 1 5FB1F628
-P 4800 1250
-F 0 "#PWR0123" H 4800 1100 50  0001 C CNN
-F 1 "+5V" V 4815 1378 50  0000 L CNN
-F 2 "" H 4800 1250 50  0001 C CNN
-F 3 "" H 4800 1250 50  0001 C CNN
-	1    4800 1250
+P 4750 1100
+F 0 "#PWR0123" H 4750 950 50  0001 C CNN
+F 1 "+5V" V 4765 1228 50  0000 L CNN
+F 2 "" H 4750 1100 50  0001 C CNN
+F 3 "" H 4750 1100 50  0001 C CNN
+	1    4750 1100
 	0    1    1    0
 $EndComp
@@
 L Device:R R3
 U 1 1 5FB20918
-P 4350 1250
-F 0 "R3" V 4143 1250 50  0000 C CNN
-F 1 "330" V 4234 1250 50  0000 C CNN
-F 2 "Resistors_SMD:R_0805_HandSoldering" V 4280 1250 50  0001 C CNN
-F 3 "~" H 4350 1250 50  0001 C CNN
-	1    4350 1250
+P 4300 1100
+F 0 "R3" V 4093 1100 50  0000 C CNN
+F 1 "150" V 4184 1100 50  0000 C CNN
+F 2 "Resistors_SMD:R_0805_HandSoldering" V 4230 1100 50  0001 C CNN
+F 3 "~" H 4300 1100 50  0001 C CNN
+	1    4300 1100
 	0    1    1    0
 $EndComp
@@
 L power:GND #PWR0124
 U 1 1 5FB225E4
-P 3900 1250
-F 0 "#PWR0124" H 3900 1000 50  0001 C CNN
-F 1 "GND" V 3905 1122 50  0000 R CNN
-F 2 "" H 3900 1250 50  0001 C CNN
-F 3 "" H 3900 1250 50  0001 C CNN
-	1    3900 1250
+P 3850 1100
+F 0 "#PWR0124" H 3850 850 50  0001 C CNN
+F 1 "GND" V 3855 972 50  0000 R CNN
+F 2 "" H 3850 1100 50  0001 C CNN
+F 3 "" H 3850 1100 50  0001 C CNN
+	1    3850 1100
 	0    1    1    0
 $EndComp
 Text Notes 4400 750  2    50   ~ 0
 LEDS
+$Comp
+L Device:LED D?
+U 1 1 5F9074FA
+P 4000 1450
+F 0 "D?" H 3993 1666 50  0000 C CNN
+F 1 "RELAY" H 3993 1575 50  0000 C CNN
+F 2 "LED_SMD:LED_1206_3216Metric_Pad1.42x1.75mm_HandSolder" H 4000 1450 50  0001 C CNN
+F 3 "~" H 4000 1450 50  0001 C CNN
+	1    4000 1450
+	1    0    0    -1
+$EndComp
+$Comp
+L Device:R R?
+U 1 1 5F9076A8
+P 4300 1450
+F 0 "R?" V 4093 1450 50  0000 C CNN
+F 1 "51" V 4184 1450 50  0000 C CNN
+F 2 "Resistors_SMD:R_0805_HandSoldering" V 4230 1450 50  0001 C CNN
+F 3 "~" H 4300 1450 50  0001 C CNN
+	1    4300 1450
+	0    1    1    0
+$EndComp
+$Comp
+L Jumper:SolderJumper_2_Open JP?
+U 1 1 5F907C26
+P 4600 1450
+F 0 "JP?" H 4600 1563 50  0000 C CNN
+F 1 "PLJP" H 4600 1564 50  0001 C CNN
+F 2 "Jumper:SolderJumper-2_P1.3mm_Open_RoundedPad1.0x1.5mm" H 4600 1450 50  0001 C CNN
+F 3 "~" H 4600 1450 50  0001 C CNN
+	1    4600 1450
+	1    0    0    -1
+$EndComp
+$Comp
+L power:GND #PWR?
+U 1 1 5F908647
+P 3850 1450
+F 0 "#PWR?" H 3850 1200 50  0001 C CNN
+F 1 "GND" V 3855 1322 50  0000 R CNN
+F 2 "" H 3850 1450 50  0001 C CNN
+F 3 "" H 3850 1450 50  0001 C CNN
+	1    3850 1450
+	0    1    1    0
+$EndComp
+Text GLabel 4750 1450 2    50   Output ~ 0
+RELAY_TRIGGER
 $EndSCHEMATC

Commit message: esp breakout
Parts:
- removed J6, J7: Conn_01x19, Pin_Headers:Pin_Header_Straight_1x19_Pitch2.54mm, symbol Connector_Generic:Conn_01x19
- removed J8: I2C, Pin_Headers:Pin_Header_Straight_1x04_Pitch2.54mm, symbol Connector_Generic:Conn_01x04
- added J3: UNK, Connectors_Phoenix:PhoenixContact_MCV-G_03x3.81mm_Vertical, symbol Connector_Generic:Conn_01x03
- added J7: GROVE_I2C, Connectors_JST:JST_PH_S5B-PH-K_05x2.00mm_Angled, symbol Connector:Conn_01x05_Male
- added JP10, JP11, JP12, JP13, JP8, JP9: Jumper_3_Open, Jumper:SolderJumper-3_P1.3mm_Open_Pad1.0x1.5mm, symbol Jumper:Jumper_3_Open
- added JP14, JP3, JP5: SolderJumper_2_Open, Jumper:SolderJumper-2_P1.3mm_Open_TrianglePad1.0x1.5mm, symbol Jumper:SolderJumper_2_Open
- added JP4, JP6, JP7: D, Jumper:SolderJumper-2_P1.3mm_Open_TrianglePad1.0x1.5mm, symbol Jumper:SolderJumper_2_Open
- added U1: ESP32-38pins, drz-lib:esp32 38pin azdelivery, symbol drz-symbols:ESP32-38pins
- J1: footprint Pin_Headers:Pin_Header_Straight_1x03_Pitch2.54mm -> Connectors_Phoenix:PhoenixContact_MCV-G_03x3.81mm_Vertical
- J2: renamed from J4; footprint Pin_Headers:Pin_Header_Straight_1x03_Pitch2.54mm -> Connectors_Phoenix:PhoenixContact_MCV-G_03x3.81mm_Vertical
- J4: renamed from J2; footprint Pin_Headers:Pin_Header_Straight_1x03_Pitch2.54mm -> Connectors_Phoenix:PhoenixContact_MCV-G_03x3.81mm_Vertical
- J5: renamed from J3; footprint Pin_Headers:Pin_Header_Straight_1x03_Pitch2.54mm -> Connectors_Phoenix:PhoenixContact_MCV-G_03x3.81mm_Vertical
- J6: renamed from J5; footprint Pin_Headers:Pin_Header_Straight_1x03_Pitch2.54mm -> Connectors_Phoenix:PhoenixContact_MCV-G_03x3.81mm_Vertical
- gave numbers to parts that had none: 3
- renumbered J9 to J8
Connections:
- net +3V3: now also J7.3 (Pin_3), JP10.3 (B), JP11.3 (B), JP12.3 (B), JP13.3 (B), JP8.3 (B), JP9.3 (B), U1.1 (3V3)
- net +5V: now also J7.1 (Pin_1), JP10.1 (A), JP11.1 (A), JP12.1 (A), JP13.1 (A), JP8.1 (A), JP9.1 (A), U1.19 (5V); no longer J4.1 (Pin_1)
- net CURRENT_SENSOR: now also JP6.1 (A); no longer J5.2 (Pin_2)
- net GND: now also J3.3 (Pin_3), J7.2 (Pin_2), U1.14 (GND), U1.20 (GND), U1.26 (GND)
- net GPIO0: now also U1.33 (GPIO0)
- net LEDMATRIX: now also U1.9 (GPIO25)
- net LED_DATA: now also JP5.2 (B); no longer J2.2 (Pin_2)
- net RELAY_TRIGGER: now also JP7.1 (A); no longer J6.2 (Pin_2)
- net SCL: now also J7.5 (Pin_5), U1.22 (GPIO22)
- net SDA: now also J7.4 (Pin_4), U1.25 (GPIO21)
- net TEMP_SENSOR: now also JP3.2 (B); no longer J1.2 (Pin_2)
- net at J4.2 (Pin_2): now also JP4.2 (B)
- net at J5.1 (Pin_1): now also JP10.2 (C)
- net at J6.1 (Pin_1): now also JP12.2 (C)
- net at J2.1 (Pin_1): now also JP11.2 (C)
- net at J1.1 (Pin_1): now also JP8.2 (C)
- new net: J4.1 (Pin_1), JP9.2 (C)
- new net: J5.2 (Pin_2), JP6.2 (B)
- new net: J6.2 (Pin_2), JP7.2 (B)
- new net: J2.2 (Pin_2), JP5.1 (A)
- new net: J1.2 (Pin_2), JP3.1 (A)
- new net: J3.1 (Pin_1), JP13.2 (C)
- new net: J3.2 (Pin_2), JP14.1 (A)
- no-connect marks 0 -> 3
Other:
- note removed: "ESP32"
- moved on the sheet: H1, H2, H3, H4, J1, J2, J4, J5, J6, J8
